File: active_filter/active_filter.sch (KiCad schematic (older format))
At the start: 16 parts, among them J1 Screw_Terminal_01x03, J2 Screw_Terminal_01x02, U1 ADA4610-2

Commit message: swapped op updated BoM
Parts:
- removed C0: 100n, default-footprints:C_0603_1608Metric, symbol Device:C_Small
- C1: value 1.2n -> 2.2n
- C2: value 1.2n -> 220p
- R1: value 18k -> 47k
- U1: value ADA4610-2 -> ADA4062-2
Connections:
- wire segments 59 -> 58
Changed lines of the file:
@@
 P 7550 2100
 F 0 "U1" H 7550 2467 50  0000 C CNN
-F 1 "ADA4610-2" H 7550 2376 50  0000 C CNN
+F 1 "ADA4062-2" H 7550 2376 50  0000 C CNN
 F 2 "default-footprints:SOIC-8_3.9x4.9mm_P1.27mm" H 7550 2100 50  0001 C CNN
 F 3 "~" H 7550 2100 50  0001 C CNN
@@
 P 7850 4500
 F 0 "U1" H 7850 4867 50  0000 C CNN
-F 1 "ADA4610-2" H 7850 4776 50  0000 C CNN
+F 1 "ADA4062-2" H 7850 4776 50  0000 C CNN
 F 2 "default-footprints:SOIC-8_3.9x4.9mm_P1.27mm" H 7850 4500 50  0001 C CNN
 F 3 "~" H 7850 4500 50  0001 C CNN
@@
 P 5750 2000
 F 0 "U1" H 5708 2046 50  0000 L CNN
-F 1 "ADA4610-2" H 5708 1955 50  0000 L CNN
+F 1 "ADA4062-2" H 5708 1955 50  0000 L CNN
 F 2 "default-footprints:SOIC-8_3.9x4.9mm_P1.27mm" H 5750 2000 50  0001 C CNN
 F 3 "~" H 5750 2000 50  0001 C CNN
@@
 P 6250 4400
 F 0 "R1" V 6457 4400 50  0000 C CNN
-F 1 "18k" V 6366 4400 50  0000 C CNN
+F 1 "47k" V 6366 4400 50  0000 C CNN
 F 2 "default-footprints:R_0603_1608Metric" V 6180 4400 50  0001 C CNN
 F 3 "~" H 6250 4400 50  0001 C CNN
@@
 P 7650 3950
 F 0 "C1" V 7421 3950 50  0000 C CNN
-F 1 "1.2n" V 7512 3950 50  0000 C CNN
+F 1 "2.2n" V 7512 3950 50  0000 C CNN
 F 2 "default-footprints:C_0603_1608Metric" H 7650 3950 50  0001 C CNN
 F 3 "~" H 7650 3950 50  0001 C CNN
@@
 P 7200 4600
 F 0 "C2" H 7292 4646 50  0000 L CNN
-F 1 "1.2n" H 7292 4555 50  0000 L CNN
+F 1 "220p" H 7292 4555 50  0000 L CNN
 F 2 "default-footprints:C_0603_1608Metric" H 7200 4600 50  0001 C CNN
 F 3 "~" H 7200 4600 50  0001 C CNN
@@
 Text GLabel 5500 4400 0    50   Input ~ 0
 IN
-Wire Wire Line
-	6100 4400 5950 4400
 $Comp
 L Device:CP_Small C10
@@
 Wire Wire Line
 	2300 2400 2550 2400
-$Comp
-L Device:C_Small C0
-U 1 1 5B75AE68
-P 5850 4400
-F 0 "C0" V 5621 4400 50  0000 C CNN
-F 1 "100n" V 5712 4400 50  0000 C CNN
-F 2 "default-footprints:C_0603_1608Metric" H 5850 4400 50  0001 C CNN
-F 3 "~" H 5850 4400 50  0001 C CNN
-	1    5850 4400
-	0    1    1    0
-$EndComp
-Wire Wire Line
-	5750 4400 5500 4400
 Wire Wire Line
 	2000 1600 2550 1600
+Wire Wire Line
+	5500 4400 6100 4400
 $EndSCHEMATC

Commit message: swapped some connectors added jumper
Parts:
- removed C12: 100n, default-footprints:C_0603_1608Metric, symbol Device:C_Small
- removed J1: Screw_Terminal_01x03, default-footprints:PinHeader_1x03_P2.54mm_Vertical_SMD_Pin1Right, symbol Connector:Screw_Terminal_01x03
- removed J2: Screw_Terminal_01x02, default-footprints:PinHeader_1x02_P2.54mm_Vertical_SMD_Pin1Right, symbol Connector:Screw_Terminal_01x02
- added J0, J1: Conn_01x03_MountingPin, symbol Connector_Generic_MountingPin:Conn_01x03_MountingPin
- added Jump0: Jumper_3_Bridged12, symbol Jumper:Jumper_3_Bridged12
Connections:
- net labels added: COM, VCC, VEE
- net labels removed: +10V
Changed lines of the file:
@@
 Wire Wire Line
 	5650 1500 5650 1700
-Wire Wire Line
-	6750 1500 8200 1500
-Connection ~ 6750 1500
 Text GLabel 8450 2100 2    50   Input ~ 0
 REF
-$Comp
-L power:+10V #PWR0101
-U 1 1 5B7312CD
-P 6750 1350
-F 0 "#PWR0101" H 6750 1200 50  0001 C CNN
-F 1 "+10V" H 6765 1523 50  0000 C CNN
-F 2 "" H 6750 1350 50  0001 C CNN
-F 3 "" H 6750 1350 50  0001 C CNN
-	1    6750 1350
-	1    0    0    -1
-$EndComp
-$Comp
-L power:GND #PWR0102
-U 1 1 5B7313CC
-P 6750 2850
-F 0 "#PWR0102" H 6750 2600 50  0001 C CNN
-F 1 "GND" H 6755 2677 50  0000 C CNN
-F 2 "" H 6750 2850 50  0001 C CNN
-F 3 "" H 6750 2850 50  0001 C CNN
-	1    6750 2850
-	1    0    0    -1
-$EndComp
 Wire Wire Line
 	6750 2700 6750 2850
 Wire Wire Line
-	6750 1350 6750 1500
-Wire Wire Line
 	7900 2100 8200 2100
 Wire Wire Line
@@
 Wire Wire Line
 	5650 2300 5650 2700
-$Comp
-L Device:C_Small C12
-U 1 1 5B732BFE
-P 8200 1750
-F 0 "C12" H 8292 1796 50  0000 L CNN
-F 1 "100n" H 8292 1705 50  0000 L CNN
-F 2 "default-footprints:C_0603_1608Metric" H 8200 1750 50  0001 C CNN
-F 3 "~" H 8200 1750 50  0001 C CNN
-	1    8200 1750
-	1    0    0    -1
-$EndComp
 $Comp
 L Device:C_Small C13
@@
 Wire Wire Line
 	6350 2700 5650 2700
-Wire Wire Line
-	8200 1650 8200 1500
-Wire Wire Line
-	8200 1850 8200 2100
 Connection ~ 8200 2100
 Wire Wire Line
@@
 	7200 4400 7550 4400
 Text GLabel 7050 5100 0    50   Input ~ 0
-REF
+COM
 Wire Wire Line
 	7200 4700 7200 5100
@@
 	1    0    0    -1
 $EndComp
-$Comp
-L Connector:Screw_Terminal_01x03 J1
-U 1 1 5B74B292
+Wire Wire Line
+	2000 1550 2000 1600
+Wire Wire Line
+	2000 1850 2000 1950
+Wire Wire Line
+	2550 1600 2550 1750
+Connection ~ 2000 1600
+Wire Wire Line
+	2000 1600 2000 1650
+Wire Wire Line
+	2550 1850 2000 1850
+Connection ~ 2000 1850
+Text GLabel 2200 2700 0    50   Input ~ 0
+IN
+Wire Wire Line
+	2500 2700 2200 2700
+Text GLabel 2250 2800 0    50   Input ~ 0
+COM
+Text GLabel 2250 2900 0    50   Input ~ 0
+OUT
+Wire Wire Line
+	2250 2800 2500 2800
+Wire Wire Line
+	2250 2900 2500 2900
+Wire Wire Line
+	2000 1600 2550 1600
+Wire Wire Line
+	5500 4400 6100 4400
+$Comp
+L Connector_Generic_MountingPin:Conn_01x03_MountingPin J0
+U 1 1 5BA57A78
 P 2750 1850
-F 0 "J1" H 2830 1892 50  0000 L CNN
-F 1 "Screw_Terminal_01x03" H 2830 1801 50  0000 L CNN
-F 2 "default-footprints:PinHeader_1x03_P2.54mm_Vertical_SMD_Pin1Right" H 2750 1850 50  0001 C CNN
+F 0 "J0" H 2837 1816 50  0000 L CNN
+F 1 "Conn_01x03_MountingPin" H 2837 1725 50  0000 L CNN
+F 2 "" H 2750 1850 50  0001 C CNN
 F 3 "~" H 2750 1850 50  0001 C CNN
 	1    2750 1850
@@
 $EndComp
 $Comp
-L Connector:Screw_Terminal_01x02 J2
-U 1 1 5B74B480
-P 2750 2300
-F 0 "J2" H 2830 2292 50  0000 L CNN
-F 1 "Screw_Terminal_01x02" H 2830 2201 50  0000 L CNN
-F 2 "default-footprints:PinHeader_1x02_P2.54mm_Vertical_SMD_Pin1Right" H 2750 2300 50  0001 C CNN
-F 3 "~" H 2750 2300 50  0001 C CNN
-	1    2750 2300
-	1    0    0    -1
-$EndComp
-$Comp
-L power:GND #PWR0103
-U 1 1 5B74DF8F
+L power:VEE #PWR?
+U 1 1 5BA5808C
+P 6750 2850
+F 0 "#PWR?" H 6750 2700 50  0001 C CNN
+F 1 "VEE" H 6768 3023 50  0000 C CNN
+F 2 "" H 6750 2850 50  0001 C CNN
+F 3 "" H 6750 2850 50  0001 C CNN
+	1    6750 2850
+	-1   0    0    1
+$EndComp
+$Comp
+L power:VCC #PWR?
+U 1 1 5BA5AA61
+P 6750 1350
+F 0 "#PWR?" H 6750 1200 50  0001 C CNN
+F 1 "VCC" H 6767 1523 50  0000 C CNN
+F 2 "" H 6750 1350 50  0001 C CNN
+F 3 "" H 6750 1350 50  0001 C CNN
+	1    6750 1350
+	1    0    0    -1
+$EndComp
+Wire Wire Line
+	6750 1350 6750 1500
+Connection ~ 6750 1500
+$Comp
+L power:VCC #PWR?
+U 1 1 5BA5B9F6
+P 2000 1550
+F 0 "#PWR?" H 2000 1400 50  0001 C CNN
+F 1 "VCC" H 2017 1723 50  0000 C CNN
+F 2 "" H 2000 1550 50  0001 C CNN
+F 3 "" H 2000 1550 50  0001 C CNN
+	1    2000 1550
+	1    0    0    -1
+$EndComp
+$Comp
+L power:VEE #PWR?
+U 1 1 5BA5C8A2
 P 2000 1950
-F 0 "#PWR0103" H 2000 1700 50  0001 C CNN
-F 1 "GND" H 2005 1777 50  0000 C CNN
+F 0 "#PWR?" H 2000 1800 50  0001 C CNN
+F 1 "VEE" H 2018 2123 50  0000 C CNN
 F 2 "" H 2000 1950 50  0001 C CNN
 F 3 "" H 2000 1950 50  0001 C CNN
 	1    2000 1950
-	1    0    0    -1
-$EndComp
-$Comp
-L power:+10V #PWR0104
-U 1 1 5B74E993
-P 2000 1550
-F 0 "#PWR0104" H 2000 1400 50  0001 C CNN
-F 1 "+10V" H 2015 1723 50  0000 C CNN
-F 2 "" H 2000 1550 50  0001 C CNN
-F 3 "" H 2000 1550 50  0001 C CNN
-	1    2000 1550
-	1    0    0    -1
-$EndComp
-Wire Wire Line
-	2000 1550 2000 1600
-Wire Wire Line
-	2000 1850 2000 1950
-Wire Wire Line
-	2550 1600 2550 1750
-Connection ~ 2000 1600
-Wire Wire Line
-	2000 1600 2000 1650
-Wire Wire Line
-	2550 1850 2000 1850
-Connection ~ 2000 1850
-Text GLabel 2250 1950 0    50   Input ~ 0
-IN
-Wire Wire Line
-	2550 1950 2250 1950
-Text GLabel 2300 2300 0    50   Input ~ 0
-OUT
-Text GLabel 2300 2400 0    50   Input ~ 0
+	-1   0    0    1
+$EndComp
+$Comp
+L power:GND #PWR?
+U 1 1 5BA5F576
+P 2400 1950
+F 0 "#PWR?" H 2400 1700 50  0001 C CNN
+F 1 "GND" H 2405 1777 50  0000 C CNN
+F 2 "" H 2400 1950 50  0001 C CNN
+F 3 "" H 2400 1950 50  0001 C CNN
+	1    2400 1950
+	1    0    0    -1
+$EndComp
+Wire Wire Line
+	2550 1950 2400 1950
+$Comp
+L Jumper:Jumper_3_Bridged12 Jump0
+U 1 1 5BA605C1
+P 2850 3750
+F 0 "Jump0" H 2850 3954 50  0000 C CNN
+F 1 "Jumper_3_Bridged12" H 2850 3863 50  0000 C CNN
+F 2 "" H 2850 3750 50  0001 C CNN
+F 3 "~" H 2850 3750 50  0001 C CNN
+	1    2850 3750
+	1    0    0    -1
+$EndComp
+Text GLabel 3100 3750 2    50   Input ~ 0
 REF
-Wire Wire Line
-	2300 2300 2550 2300
-Wire Wire Line
-	2300 2400 2550 2400
-Wire Wire Line
-	2000 1600 2550 1600
-Wire Wire Line
-	5500 4400 6100 4400
+Text GLabel 2850 3900 3    50   Input ~ 0
+COM
+$Comp
+L power:GND #PWR?
+U 1 1 5BA614F9
+P 2450 3800
+F 0 "#PWR?" H 2450 3550 50  0001 C CNN
+F 1 "GND" H 2455 3627 50  0000 C CNN
+F 2 "" H 2450 3800 50  0001 C CNN
+F 3 "" H 2450 3800 50  0001 C CNN
+	1    2450 3800
+	1    0    0    -1
+$EndComp
+Wire Wire Line
+	2450 3800 2450 3750
+Wire Wire Line
+	2450 3750 2600 3750
+$Comp
+L Connector_Generic_MountingPin:Conn_01x03_MountingPin J1
+U 1 1 5BA6345F
+P 2700 2800
+F 0 "J1" H 2787 2766 50  0000 L CNN
+F 1 "Conn_01x03_MountingPin" H 2787 2675 50  0000 L CNN
+F 2 "" H 2700 2800 50  0001 C CNN
+F 3 "~" H 2700 2800 50  0001 C CNN
+	1    2700 2800
+	1    0    0    -1
+$EndComp
 $EndSCHEMATC

Commit message: changed parts checked design rules
Parts:
- J0, J1, Jump0: footprint (none) -> default-footprints:PinHeader_1x03_P2.54mm_Vertical
- RV4: footprint default-footprints:Potentiometer_Vishay_TS53YL_Vertical -> default-footprints:Potentiometer_Bourns_PTV09A-1_Single_Vertical
Changed lines of the file:
@@
 F 0 "RV4" H 8180 4896 50  0000 R CNN
 F 1 "100k" H 8180 4805 50  0000 R CNN
-F 2 "default-footprints:Potentiometer_Vishay_TS53YL_Vertical" H 8250 4850 50  0001 C CNN
+F 2 "default-footprints:Potentiometer_Bourns_PTV09A-1_Single_Vertical" H 8250 4850 50  0001 C CNN
 F 3 "~" H 8250 4850 50  0001 C CNN
 	1    8250 4850
@@
 F 0 "J0" H 2837 1816 50  0000 L CNN
 F 1 "Conn_01x03_MountingPin" H 2837 1725 50  0000 L CNN
-F 2 "" H 2750 1850 50  0001 C CNN
+F 2 "default-footprints:PinHeader_1x03_P2.54mm_Vertical" H 2750 1850 50  0001 C CNN
 F 3 "~" H 2750 1850 50  0001 C CNN
 	1    2750 1850
@@
 $EndComp
 $Comp
-L power:VEE #PWR?
+L power:VEE #PWR0101
 U 1 1 5BA5808C
 P 6750 2850
-F 0 "#PWR?" H 6750 2700 50  0001 C CNN
+F 0 "#PWR0101" H 6750 2700 50  0001 C CNN
 F 1 "VEE" H 6768 3023 50  0000 C CNN
 F 2 "" H 6750 2850 50  0001 C CNN
@@
 $EndComp
 $Comp
-L power:VCC #PWR?
+L power:VCC #PWR0102
 U 1 1 5BA5AA61
 P 6750 1350
-F 0 "#PWR?" H 6750 1200 50  0001 C CNN
+F 0 "#PWR0102" H 6750 1200 50  0001 C CNN
 F 1 "VCC" H 6767 1523 50  0000 C CNN
 F 2 "" H 6750 1350 50  0001 C CNN
@@
 Connection ~ 6750 1500
 $Comp
-L power:VCC #PWR?
+L power:VCC #PWR0103
 U 1 1 5BA5B9F6
 P 2000 1550
-F 0 "#PWR?" H 2000 1400 50  0001 C CNN
+F 0 "#PWR0103" H 2000 1400 50  0001 C CNN
 F 1 "VCC" H 2017 1723 50  0000 C CNN
 F 2 "" H 2000 1550 50  0001 C CNN
@@
 $EndComp
 $Comp
-L power:VEE #PWR?
+L power:VEE #PWR0104
 U 1 1 5BA5C8A2
 P 2000 1950
-F 0 "#PWR?" H 2000 1800 50  0001 C CNN
+F 0 "#PWR0104" H 2000 1800 50  0001 C CNN
 F 1 "VEE" H 2018 2123 50  0000 C CNN
 F 2 "" H 2000 1950 50  0001 C CNN
@@
 $EndComp
 $Comp
-L power:GND #PWR?
+L power:GND #PWR0105
 U 1 1 5BA5F576
 P 2400 1950
-F 0 "#PWR?" H 2400 1700 50  0001 C CNN
+F 0 "#PWR0105" H 2400 1700 50  0001 C CNN
 F 1 "GND" H 2405 1777 50  0000 C CNN
 F 2 "" H 2400 1950 50  0001 C CNN
@@
 F 0 "Jump0" H 2850 3954 50  0000 C CNN
 F 1 "Jumper_3_Bridged12" H 2850 3863 50  0000 C CNN
-F 2 "" H 2850 3750 50  0001 C CNN
+F 2 "default-footprints:PinHeader_1x03_P2.54mm_Vertical" H 2850 3750 50  0001 C CNN
 F 3 "~" H 2850 3750 50  0001 C CNN
 	1    2850 3750
@@
 COM
 $Comp
-L power:GND #PWR?
+L power:GND #PWR0106
 U 1 1 5BA614F9
 P 2450 3800
-F 0 "#PWR?" H 2450 3550 50  0001 C CNN
+F 0 "#PWR0106" H 2450 3550 50  0001 C CNN
 F 1 "GND" H 2455 3627 50  0000 C CNN
 F 2 "" H 2450 3800 50  0001 C CNN
@@
 F 0 "J1" H 2787 2766 50  0000 L CNN
 F 1 "Conn_01x03_MountingPin" H 2787 2675 50  0000 L CNN
-F 2 "" H 2700 2800 50  0001 C CNN
+F 2 "default-footprints:PinHeader_1x03_P2.54mm_Vertical" H 2700 2800 50  0001 C CNN
 F 3 "~" H 2700 2800 50  0001 C CNN
 	1    2700 2800

Commit message: added power_flag symbols
Connections:
- wire segments 58 -> 63
Changed lines of the file:
@@
 	1    0    0    -1
 $EndComp
+$Comp
+L power:PWR_FLAG #FLG?
+U 1 1 5BA91C30
+P 1800 1550
+F 0 "#FLG?" H 1800 1625 50  0001 C CNN
+F 1 "PWR_FLAG" H 1800 1724 50  0000 C CNN
+F 2 "" H 1800 1550 50  0001 C CNN
+F 3 "~" H 1800 1550 50  0001 C CNN
+	1    1800 1550
+	1    0    0    -1
+$EndComp
+$Comp
+L power:PWR_FLAG #FLG?
+U 1 1 5BA91CC9
+P 1800 1950
+F 0 "#FLG?" H 1800 2025 50  0001 C CNN
+F 1 "PWR_FLAG" H 1800 2123 50  0000 C CNN
+F 2 "" H 1800 1950 50  0001 C CNN
+F 3 "~" H 1800 1950 50  0001 C CNN
+	1    1800 1950
+	-1   0    0    1
+$EndComp
+$Comp
+L power:PWR_FLAG #FLG?
+U 1 1 5BA91D40
+P 2250 1950
+F 0 "#FLG?" H 2250 2025 50  0001 C CNN
+F 1 "PWR_FLAG" H 2250 2123 50  0000 C CNN
+F 2 "" H 2250 1950 50  0001 C CNN
+F 3 "~" H 2250 1950 50  0001 C CNN
+	1    2250 1950
+	-1   0    0    1
+$EndComp
+Wire Wire Line
+	1800 1550 1800 1600
+Wire Wire Line
+	1800 1600 2000 1600
+Wire Wire Line
+	1800 1950 1800 1850
+Wire Wire Line
+	1800 1850 2000 1850
+Wire Wire Line
+	2250 1950 2400 1950
+Connection ~ 2400 1950
 $EndSCHEMATC

Commit message: added second decoupling cap and swapped symbols
Parts:
- added C12: 10u, default-footprints:CP_Elec_5x5.4, symbol Device:CP_Small
- J0: value Conn_01x03_MountingPin -> Conn_01x03; symbol Connector_Generic_MountingPin:Conn_01x03_MountingPin -> Connector:Conn_01x03_Male
- J1: symbol Connector_Generic_MountingPin:Conn_01x03_MountingPin -> Connector:Conn_01x03_Male
Connections:
- wire segments 63 -> 68
Changed lines of the file:
@@
 L Device:CP_Small C10
 U 1 1 5B7443C5
-P 2000 1750
-F 0 "C10" H 2088 1796 50  0000 L CNN
-F 1 "10u" H 2088 1705 50  0000 L CNN
-F 2 "default-footprints:CP_Elec_5x5.4" H 2000 1750 50  0001 C CNN
-F 3 "~" H 2000 1750 50  0001 C CNN
-	1    2000 1750
-	1    0    0    -1
-$EndComp
-Wire Wire Line
-	2000 1550 2000 1600
-Wire Wire Line
-	2000 1850 2000 1950
-Wire Wire Line
-	2550 1600 2550 1750
-Connection ~ 2000 1600
-Wire Wire Line
-	2000 1600 2000 1650
-Wire Wire Line
-	2550 1850 2000 1850
-Connection ~ 2000 1850
+P 2250 1950
+F 0 "C10" H 2338 1996 50  0000 L CNN
+F 1 "10u" H 2338 1905 50  0000 L CNN
+F 2 "default-footprints:CP_Elec_5x5.4" H 2250 1950 50  0001 C CNN
+F 3 "~" H 2250 1950 50  0001 C CNN
+	1    2250 1950
+	1    0    0    -1
+$EndComp
+Wire Wire Line
+	2000 1400 2000 1450
+Wire Wire Line
+	1950 2100 1950 2200
+Connection ~ 2000 1450
 Text GLabel 2200 2700 0    50   Input ~ 0
 IN
@@
 	2250 2900 2500 2900
 Wire Wire Line
-	2000 1600 2550 1600
+	2000 1450 2250 1450
 Wire Wire Line
 	5500 4400 6100 4400
 $Comp
-L Connector_Generic_MountingPin:Conn_01x03_MountingPin J0
+L Connector:Conn_01x03_Male J0
 U 1 1 5BA57A78
 P 2750 1850
 F 0 "J0" H 2837 1816 50  0000 L CNN
-F 1 "Conn_01x03_MountingPin" H 2837 1725 50  0000 L CNN
+F 1 "Conn_01x03" H 2837 1725 50  0000 L CNN
 F 2 "default-footprints:PinHeader_1x03_P2.54mm_Vertical" H 2750 1850 50  0001 C CNN
 F 3 "~" H 2750 1850 50  0001 C CNN
 	1    2750 1850
-	1    0    0    -1
+	-1   0    0    -1
 $EndComp
 $Comp
@@
 L power:VCC #PWR0103
 U 1 1 5BA5B9F6
-P 2000 1550
-F 0 "#PWR0103" H 2000 1400 50  0001 C CNN
-F 1 "VCC" H 2017 1723 50  0000 C CNN
-F 2 "" H 2000 1550 50  0001 C CNN
-F 3 "" H 2000 1550 50  0001 C CNN
-	1    2000 1550
+P 2000 1400
+F 0 "#PWR0103" H 2000 1250 50  0001 C CNN
+F 1 "VCC" H 2017 1573 50  0000 C CNN
+F 2 "" H 2000 1400 50  0001 C CNN
+F 3 "" H 2000 1400 50  0001 C CNN
+	1    2000 1400
 	1    0    0    -1
 $EndComp
@@
 L power:VEE #PWR0104
 U 1 1 5BA5C8A2
-P 2000 1950
-F 0 "#PWR0104" H 2000 1800 50  0001 C CNN
-F 1 "VEE" H 2018 2123 50  0000 C CNN
-F 2 "" H 2000 1950 50  0001 C CNN
-F 3 "" H 2000 1950 50  0001 C CNN
-	1    2000 1950
+P 1950 2200
+F 0 "#PWR0104" H 1950 2050 50  0001 C CNN
+F 1 "VEE" H 1968 2373 50  0000 C CNN
+F 2 "" H 1950 2200 50  0001 C CNN
+F 3 "" H 1950 2200 50  0001 C CNN
+	1    1950 2200
 	-1   0    0    1
 $EndComp
@@
 L power:GND #PWR0105
 U 1 1 5BA5F576
-P 2400 1950
-F 0 "#PWR0105" H 2400 1700 50  0001 C CNN
-F 1 "GND" H 2405 1777 50  0000 C CNN
-F 2 "" H 2400 1950 50  0001 C CNN
-F 3 "" H 2400 1950 50  0001 C CNN
-	1    2400 1950
-	1    0    0    -1
-$EndComp
-Wire Wire Line
-	2550 1950 2400 1950
+P 1950 1850
+F 0 "#PWR0105" H 1950 1600 50  0001 C CNN
+F 1 "GND" H 1955 1677 50  0000 C CNN
+F 2 "" H 1950 1850 50  0001 C CNN
+F 3 "" H 1950 1850 50  0001 C CNN
+	1    1950 1850
+	1    0    0    -1
+$EndComp
 $Comp
 L Jumper:Jumper_3_Bridged12 Jump0
@@
 	2450 3750 2600 3750
 $Comp
-L Connector_Generic_MountingPin:Conn_01x03_MountingPin J1
+L Connector:Conn_01x03_Male J1
 U 1 1 5BA6345F
 P 2700 2800
@@
 F 3 "~" H 2700 2800 50  0001 C CNN
 	1    2700 2800
-	1    0    0    -1
-$EndComp
-$Comp
-L power:PWR_FLAG #FLG?
+	-1   0    0    -1
+$EndComp
+$Comp
+L power:PWR_FLAG #FLG0101
 U 1 1 5BA91C30
-P 1800 1550
-F 0 "#FLG?" H 1800 1625 50  0001 C CNN
-F 1 "PWR_FLAG" H 1800 1724 50  0000 C CNN
-F 2 "" H 1800 1550 50  0001 C CNN
-F 3 "~" H 1800 1550 50  0001 C CNN
-	1    1800 1550
-	1    0    0    -1
-$EndComp
-$Comp
-L power:PWR_FLAG #FLG?
+P 1800 1400
+F 0 "#FLG0101" H 1800 1475 50  0001 C CNN
+F 1 "PWR_FLAG" H 1800 1574 50  0000 C CNN
+F 2 "" H 1800 1400 50  0001 C CNN
+F 3 "~" H 1800 1400 50  0001 C CNN
+	1    1800 1400
+	1    0    0    -1
+$EndComp
+$Comp
+L power:PWR_FLAG #FLG0102
 U 1 1 5BA91CC9
-P 1800 1950
-F 0 "#FLG?" H 1800 2025 50  0001 C CNN
-F 1 "PWR_FLAG" H 1800 2123 50  0000 C CNN
-F 2 "" H 1800 1950 50  0001 C CNN
-F 3 "~" H 1800 1950 50  0001 C CNN
-	1    1800 1950
-	-1   0    0    1
-$EndComp
-$Comp
-L power:PWR_FLAG #FLG?
+P 1750 2200
+F 0 "#FLG0102" H 1750 2275 50  0001 C CNN
+F 1 "PWR_FLAG" H 1750 2373 50  0000 C CNN
+F 2 "" H 1750 2200 50  0001 C CNN
+F 3 "~" H 1750 2200 50  0001 C CNN
+	1    1750 2200
+	-1   0    0    1
+$EndComp
+$Comp
+L power:PWR_FLAG #FLG0103
 U 1 1 5BA91D40
-P 2250 1950
-F 0 "#FLG?" H 2250 2025 50  0001 C CNN
-F 1 "PWR_FLAG" H 2250 2123 50  0000 C CNN
-F 2 "" H 2250 1950 50  0001 C CNN
-F 3 "~" H 2250 1950 50  0001 C CNN
-	1    2250 1950
-	-1   0    0    1
-$EndComp
-Wire Wire Line
-	1800 1550 1800 1600
-Wire Wire Line
-	1800 1600 2000 1600
-Wire Wire Line
-	1800 1950 1800 1850
-Wire Wire Line
-	1800 1850 2000 1850
-Wire Wire Line
-	2250 1950 2400 1950
-Connection ~ 2400 1950
+P 1800 1850
+F 0 "#FLG0103" H 1800 1925 50  0001 C CNN
+F 1 "PWR_FLAG" H 1800 2023 50  0000 C CNN
+F 2 "" H 1800 1850 50  0001 C CNN
+F 3 "~" H 1800 1850 50  0001 C CNN
+	1    1800 1850
+	-1   0    0    1
+$EndComp
+Wire Wire Line
+	1800 1400 1800 1450
+Wire Wire Line
+	1800 1450 2000 1450
+Wire Wire Line
+	1750 2200 1750 2100
+$Comp
+L Device:CP_Small C12
+U 1 1 5BAA18A4
+P 2250 1550
+F 0 "C12" H 2338 1596 50  0000 L CNN
+F 1 "10u" H 2338 1505 50  0000 L CNN
+F 2 "default-footprints:CP_Elec_5x5.4" H 2250 1550 50  0001 C CNN
+F 3 "~" H 2250 1550 50  0001 C CNN
+	1    2250 1550
+	1    0    0    -1
+$EndComp
+Connection ~ 2250 1450
+Wire Wire Line
+	2250 1450 2550 1450
+Connection ~ 1950 2100
+Wire Wire Line
+	2550 1850 2250 1850
+Wire Wire Line
+	2250 1850 1950 1850
+Connection ~ 2250 1850
+Wire Wire Line
+	1950 1850 1800 1850
+Connection ~ 1950 1850
+Wire Wire Line
+	1750 2100 1950 2100
+Wire Wire Line
+	1950 2100 2250 2100
+Wire Wire Line
+	2550 1950 2550 2100
+Wire Wire Line
+	2250 2050 2250 2100
+Connection ~ 2250 2100
+Wire Wire Line
+	2250 2100 2550 2100
+Wire Wire Line
+	2550 1450 2550 1750
+Wire Wire Line
+	2250 1650 2250 1850
 $EndSCHEMATC
